File: datasheets/slave.kicad_pcb (KiCad board)
At the start: 2 copper layers, 71.1 x 50.8 mm, 20 parts, among them J1 Screw_Terminal_1x02, J2 Screw_Terminal_1x03, Q1 IRFU9024N, Q2 IRFU9024N, Q3 IRFU9024N, U1 PC817, U2 PC817, U3 PC817

Commit message: Исправление ошибок в схемах
Parts:
- added C1: C, Capacitors_THT:C_Disc_D6.0mm_W2.5mm_P5.00mm, F.Cu at (241.3, 63.5)
- added C2: CP, w_capacitors:CP_5x11mm, F.Cu at (226.1, 56.9)
- added J3: Screw_Terminal_1x02, w_conn_screw:mors_2p, F.Cu at (233.7, 53.3)
- added U4: nRF24L01, nRF24x:nRF24L01-NA, F.Cu at (215.3, 67.3)
- added U5: Arduino_Nano, arduino:ArduinoNano, F.Cu at (198.1, 73.6)
- added U6: KA378R33, TO_SOT_Packages_THT:TO-220-4_Vertical, F.Cu at (226.1, 63.5)
- J1: footprint Connectors_Terminal_Blocks:TerminalBlock_Pheonix_MKDS1.5-2pol -> w_conn_screw:mors_2p
- J2: footprint Connectors_Terminal_Blocks:TerminalBlock_Pheonix_MKDS1.5-3pol -> w_conn_screw:mors_3p
- R1: value R -> 470; footprint Resistors_THT:R_Axial_DIN0207_L6.3mm_D2.5mm_P2.54mm_Vertical -> Resistors_THT:R_Axial_DIN0207_L6.3mm_D2.5mm_P10.16mm_Horizontal
- R2: value R -> 10k
- R3: value R -> 100
- R4, R5: footprint Resistors_THT:R_Axial_DIN0207_L6.3mm_D2.5mm_P2.54mm_Vertical -> Resistors_THT:R_Axial_DIN0207_L6.3mm_D2.5mm_P10.16mm_Horizontal
- moved J2 4.92 mm to (248.9, 71.1), turned to 270 degrees
- moved J1 2.46 mm to (248.9, 58.4), turned to 270 degrees
Connections:
- J1 pad 1: /P_VCC -> /P_GND
- J1 pad 2: /P_GND -> /P_VCC
- J2 pad 1: /OUT_3 -> /OUT_1
- J2 pad 3: /OUT_1 -> /OUT_3
- Q1 pad 2: /P_VCC -> /OUT_1
- Q1 pad 3: /OUT_1 -> /P_VCC
- Q2 pad 2: /P_VCC -> /OUT_2
- Q2 pad 3: /OUT_2 -> /P_VCC
- Q3 pad 2: /P_VCC -> /OUT_3
- Q3 pad 3: /OUT_3 -> /P_VCC
- R1 pad 2: Net-(R1-Pad2) -> /IN_1
- R4 pad 2: Net-(R4-Pad2) -> /IN_2
- R5 pad 2: Net-(R5-Pad2) -> /IN_3
- U1 pad 2: Net-(U1-Pad2) -> /D_GND
- U2 pad 2: Net-(U2-Pad2) -> /D_GND
- U3 pad 2: Net-(U3-Pad2) -> /D_GND
Routing:
- net /D_GND: track 0.00 -> 132.6 mm
- net /D_VCC: track 0.00 -> 110.1 mm
- net /IRQ: track 0.00 -> 48.6 mm
- net /SCK: track 0.00 -> 30.8 mm
- net /IN_3: track 0.00 -> 21.4 mm
- net /MOSI: track 0.00 -> 20.6 mm
- net /SCN/D9: track 0.00 -> 19.6 mm
- net /3V3: track 0.00 -> 18.9 mm
- net /CE/SS: track 0.00 -> 18.8 mm
- net /IN_2: track 0.00 -> 14.5 mm
- net /MISO: track 0.00 -> 11.2 mm
- net /IN_1: track 0.00 -> 7.62 mm
- net /P_VCC: track 59.1 -> 52.7 mm
- net /P_GND: track 73.1 -> 76.1 mm
- net /OUT_3: track 25.0 -> 22.3 mm
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Other:
- net class Power added: clearance 0.2, trace_width 1, via_dia 0.6, via_drill 0.4

Commit message: Правка схем
Parts:
- D1, D2, D3: footprint user_diodes:D_DO-41_SOD81_P12.70mm_Horizontal -> Diodes_THT:D_DO-41_SOD81_P12.70mm_Horizontal
- U5: value Arduino_Nano -> ArduinoNano; footprint arduino:ArduinoNano -> Modules:Arduino_Nano
- moved U5 19.4 mm to (205.7, 91.4), turned to 180 degrees
- moved C1 9.91 mm to (241.3, 53.6), turned to 270 degrees
Routing:
- net /D_GND: track 132.6 -> 138.5 mm
- net /D_VCC: track 110.1 -> 108.9 mm

Commit message: Добавление библиотек компонентов для KiCad.
Parts:
- moved D3 2.54 mm to (251.5, 83.8)
- moved D1 2.54 mm to (246.4, 83.8)
- moved D2 2.54 mm to (248.9, 83.8)
Routing:
- net /OUT_2: track 25.0 -> 28.6 mm
- net /OUT_3: track 22.3 -> 25.7 mm
- net /P_GND: track 76.1 -> 78.6 mm
- net /OUT_1: track 25.2 -> 26.2 mm
