File: datasheets/master/master.sch (KiCad schematic (older format))
At the start: 11 parts, among them J1 Screw_Terminal_01x03, J2 Screw_Terminal_01x03, J3 Screw_Terminal_01x03, J4 Screw_Terminal_01x03, J5 Screw_Terminal_01x03, J6 Screw_Terminal_01x02, U1 nRF24L01+PA, U2 ArduinoNano

Commit message: Обновление и добавление документации.
Parts:
- added SH?: ARDUINO_MEGA, symbol ARDUINO_MEGA
Changed lines of the file:
@@
 +3V3
 Connection ~ 4900 1300
+$Comp
+L ARDUINO_MEGA SH?
+U 1 1 5B3DA37D
+P 7000 3100
+F 0 "SH?" H 7000 3625 60  0000 C CNN
+F 1 "ARDUINO_MEGA" H 7000 3825 60  0000 C CNN
+F 2 "" H 6050 3400 60  0000 C CNN
+F 3 "" H 6050 3400 60  0000 C CNN
+	1    7000 3100
+	1    0    0    -1
+$EndComp
 $EndSCHEMATC
